Commit message: 02.01.21

File: mark1/src/mark1_description/urdf/mark1.xacro (robot description, xacro)
@@ -50,9 +50,6 @@
         value="1.483" />
       <inertia
-        ixx="0.0078938"
-        ixy="1.3747E-18"
-        ixz="-2.0644E-19"
-        iyy="0.014347"
-        iyz="-3.4936E-18"
+        ixx="0.0078938" ixy="1.3747E-18" ixz="-2.0644E-19"
+        iyy="0.014347" iyz="-3.4936E-18"
         izz="0.0078938" />
     </inertial>
@@ -113,5 +110,5 @@
       <geometry>
         <mesh
-          filename="package://mark1/src/mark1_description/meshes/Right_Motor_Joint.STL" />
+          filename="package://mark1/src/mark1_description/meshes/Right_Motor_Link.STL" />
       </geometry>
       <material
@@ -127,5 +124,5 @@
       <geometry>
         <mesh
-          filename="package://mark1/src/mark1_description/meshes/Right_Motor_Joint.STL" />
+          filename="package://mark1/src/mark1_description/meshes/Right_Motor_Link.STL" />
       </geometry>
     </collision>
@@ -142,29 +139,3 @@
       xyz="0 1 0" />
   </joint>
-  <joint name="hokuyo_joint" type="fixed">
-    <axis xyz="0 1 0" />
-    <origin xyz="-0.15 0 .18" rpy="0 0 0"/>
-    <parent link="base_link"/>
-    <child link="hokuyo"/>
-  </joint>
-  <!-- Hokuyo Laser -->
-  <link name="hokuyo">
-    <collision>
-      <origin xyz="0 0 0" rpy="0 0 0"/>
-      <geometry>
-    <box size="0.1 0.1 0.1"/>
-      </geometry>
-    </collision>
-    <visual>
-      <origin xyz="0 0 0" rpy="0 0 0"/>
-      <geometry>
-        <mesh filename="package://mark1/src/mark1_description/meshes/hokuyo.dae"/>
-      </geometry>
-    </visual>
-    <inertial>
-      <mass value="1e-5" />
-      <origin xyz="0 0 0" rpy="0 0 0"/>
-      <inertia ixx="1e-6" ixy="0" ixz="0" iyy="1e-6" iyz="0" izz="1e-6" />
-    </inertial>
-  </link>
 </robot>

Commit message: Lesson_2 Add Sensor

File: mark1/src/mark1_description/urdf/mark1.xacro (robot description, xacro)
@@ -1,6 +1,4 @@
 <?xml version='1.0'?>
 <robot name="mark1" xmlns:xacro="http://www.ros.org/wiki/xacro">
-  <xacro:property name="cameraSize" value="0.05"/>
-  <xacro:property name="cameraMass" value="0.1"/>
   <xacro:include filename="$(find mark1)/src/mark1_description/urdf/mark1.gazebo" />
   <xacro:include filename="$(find mark1)/src/mark1_description/urdf/materials.xacro" />
@@ -139,3 +137,56 @@
       xyz="0 1 0" />
   </joint>
+ <joint name="hokuyo_joint" type="fixed">
+    <axis xyz="0 1 0" />
+    <origin xyz="-0.1 0 0.19" rpy="0 0 0"/>
+    <parent link="base_link"/>
+    <child link="hokuyo_link"/>
+  </joint>
+  <!-- Hokuyo Laser -->
+  <link name="hokuyo_link">
+    <collision>
+      <origin xyz="0 0 0" rpy="0 0 0"/>
+      <geometry>
+    <box size="0.1 0.1 0.1"/>
+      </geometry>
+    </collision>
+    <visual>
+      <origin xyz="0 0 0" rpy="0 0 0"/>
+      <geometry>
+        <mesh filename="package://mark1/src/mark1_description/meshes/hokuyo.dae"/>
+      </geometry>
+    </visual>
+    <inertial>
+      <mass value="1e-5" />
+      <origin xyz="0 0 0" rpy="0 0 0"/>
+      <inertia ixx="1e-6" ixy="0" ixz="0" iyy="1e-6" iyz="0" izz="1e-6" />
+    </inertial>
+  </link>
+<joint name="camera_joint" type="fixed">
+    <axis xyz="0 1 0" />
+    <origin xyz="0.27 0 0.05" rpy="0 0  0"/>
+    <parent link="base_link"/>
+    <child link="camera_link"/>
+  </joint>
+  <!-- Camera -->
+  <link name="camera_link">
+    <collision>
+      <origin xyz="0 0 0" rpy="0 0 0"/>
+      <geometry>
+    <box size="0 0 0"/>
+      </geometry>
+    </collision>
+    <visual>
+      <origin xyz="0 0 0" rpy="0 0 0"/>
+      <geometry>
+    <box size="0.05 0.05  0.05"/>
+      </geometry>
+      <material name="red"/>
+    </visual>
+    <inertial>
+      <mass value="1e-5" />
+      <origin xyz="0 0 0" rpy="0 0 0"/>
+      <inertia ixx="1e-6" ixy="0" ixz="0" iyy="1e-6" iyz="0" izz="1e-6" />
+    </inertial>
+  </link>
 </robot>

Commit message: 03.01.21 Lesson_3 move_base V1.1

File: mark1/src/mark1_description/urdf/mark1.xacro (robot description, xacro)
@@ -141,8 +141,8 @@
     <origin xyz="-0.1 0 0.19" rpy="0 0 0"/>
     <parent link="base_link"/>
-    <child link="hokuyo_link"/>
+    <child link="hokuyo"/>
   </joint>
   <!-- Hokuyo Laser -->
-  <link name="hokuyo_link">
+  <link name="hokuyo">
     <collision>
       <origin xyz="0 0 0" rpy="0 0 0"/>

Commit message: 31.01.21 Lesson_7 DepthCamera

File: mark1/src/mark1_description/urdf/mark1.xacro (robot description, xacro)
@@ -137,5 +137,25 @@
       xyz="0 1 0" />
   </joint>
- <joint name="hokuyo_joint" type="fixed">
+  <!-- Hokuyo Laser -->
+  <link name="hokuyo">
+    <collision>
+      <origin xyz="0 0 0" rpy="0 0 0"/>
+      <geometry>
+    <box size="0.1 0.1 0.1"/>
+      </geometry>
+    </collision>
+    <visual>
+      <origin xyz="0 0 0" rpy="0 0 0"/>
+      <geometry>
+        <mesh filename="package://mark1/src/mark1_description/meshes/hokuyo.dae"/>
+      </geometry>
+    </visual>
+    <inertial>
+      <mass value="1e-5" />
+      <origin xyz="0 0 0" rpy="0 0 0"/>
+      <inertia ixx="1e-6" ixy="0" ixz="0" iyy="1e-6" iyz="0" izz="1e-6" />
+    </inertial>
+  </link>
+<joint name="hokuyo_joint" type="fixed">
     <axis xyz="0 1 0" />
     <origin xyz="-0.1 0 0.19" rpy="0 0 0"/>
@@ -143,17 +163,18 @@
     <child link="hokuyo"/>
   </joint>
-  <!-- Hokuyo Laser -->
-  <link name="hokuyo">
-    <collision>
-      <origin xyz="0 0 0" rpy="0 0 0"/>
-      <geometry>
-    <box size="0.1 0.1 0.1"/>
-      </geometry>
-    </collision>
-    <visual>
-      <origin xyz="0 0 0" rpy="0 0 0"/>
-      <geometry>
-        <mesh filename="package://mark1/src/mark1_description/meshes/hokuyo.dae"/>
-      </geometry>
+  <!-- Camera -->
+  <link name="camera_link">
+    <collision>
+      <origin xyz="0 0 0" rpy="0 0 0"/>
+      <geometry>
+    <box size="0 0 0"/>
+      </geometry>
+    </collision>
+    <visual>
+      <origin xyz="0 0 0" rpy="0 0 0"/>
+      <geometry>
+    <box size="0.05 0.05  0.05"/>
+      </geometry>
+      <material name="red"/>
     </visual>
     <inertial>
@@ -169,10 +190,10 @@
     <child link="camera_link"/>
   </joint>
-  <!-- Camera -->
-  <link name="camera_link">
-    <collision>
-      <origin xyz="0 0 0" rpy="0 0 0"/>
-      <geometry>
-    <box size="0 0 0"/>
+  	  <!-- Depth Camera -->
+<link name="depth_camera_link">
+    <collision>
+      <origin xyz="0 0 0" rpy="0 0 0"/>
+      <geometry>
+    <box size="0.05 0.05 0.05"/>
       </geometry>
     </collision>
@@ -182,11 +203,25 @@
     <box size="0.05 0.05  0.05"/>
       </geometry>
-      <material name="red"/>
-    </visual>
-    <inertial>
-      <mass value="1e-5" />
+      <material name="blue"/>
+    </visual>
+    <inertial>
+      <mass value="0.210" />
       <origin xyz="0 0 0" rpy="0 0 0"/>
       <inertia ixx="1e-6" ixy="0" ixz="0" iyy="1e-6" iyz="0" izz="1e-6" />
     </inertial>
   </link>
+<joint name="depth_camera_joint" type="fixed">
+    <axis xyz="0 1 0" />
+    <origin xyz="-0.1 0 0.4" rpy="0 0  0"/>
+    <parent link="base_link"/>
+    <child link="depth_camera_link"/>
+  </joint>
+ <link name="depth_camera_optical">
+  </link>
+ <joint name="depth_camera_optical_joint" type="fixed">
+    <axis xyz="0 1 0" />
+    <origin xyz="0 0 0" rpy="-1.57 0 -1.57"/>
+    <parent link="depth_camera_link"/>
+    <child link="depth_camera_optical"/>
+  </joint>
 </robot>

Commit message: AMCL/GMAPPING V1.3 31.05.21

File: mark1/src/mark1_description/urdf/mark1.xacro (robot description, xacro)
@@ -137,4 +137,10 @@
       xyz="0 1 0" />
   </joint>
+ <joint name="hokuyo_joint" type="fixed">
+    <axis xyz="0 1 0" />
+    <origin xyz="-0.1 0 0.19" rpy="0 0 0"/>
+    <parent link="base_link"/>
+    <child link="hokuyo"/>
+  </joint>
   <!-- Hokuyo Laser -->
   <link name="hokuyo">
@@ -157,9 +163,9 @@
     </inertial>
   </link>
-<joint name="hokuyo_joint" type="fixed">
+<joint name="camera_joint" type="fixed">
     <axis xyz="0 1 0" />
-    <origin xyz="-0.1 0 0.19" rpy="0 0 0"/>
+    <origin xyz="0.27 0 0.05" rpy="0 0  0"/>
     <parent link="base_link"/>
-    <child link="hokuyo"/>
+    <child link="camera_link"/>
   </joint>
   <!-- Camera -->
@@ -184,44 +190,3 @@
     </inertial>
   </link>
-<joint name="camera_joint" type="fixed">
-    <axis xyz="0 1 0" />
-    <origin xyz="0.27 0 0.05" rpy="0 0  0"/>
-    <parent link="base_link"/>
-    <child link="camera_link"/>
-  </joint>
-  	  <!-- Depth Camera -->
-<link name="depth_camera_link">
-    <collision>
-      <origin xyz="0 0 0" rpy="0 0 0"/>
-      <geometry>
-    <box size="0.05 0.05 0.05"/>
-      </geometry>
-    </collision>
-    <visual>
-      <origin xyz="0 0 0" rpy="0 0 0"/>
-      <geometry>
-    <box size="0.05 0.05  0.05"/>
-      </geometry>
-      <material name="blue"/>
-    </visual>
-    <inertial>
-      <mass value="0.210" />
-      <origin xyz="0 0 0" rpy="0 0 0"/>
-      <inertia ixx="1e-6" ixy="0" ixz="0" iyy="1e-6" iyz="0" izz="1e-6" />
-    </inertial>
-  </link>
-<joint name="depth_camera_joint" type="fixed">
-    <axis xyz="0 1 0" />
-    <origin xyz="-0.1 0 0.4" rpy="0 0  0"/>
-    <parent link="base_link"/>
-    <child link="depth_camera_link"/>
-  </joint>
- <link name="depth_camera_optical">
-  </link>
- <joint name="depth_camera_optical_joint" type="fixed">
-    <axis xyz="0 1 0" />
-    <origin xyz="0 0 0" rpy="-1.57 0 -1.57"/>
-    <parent link="depth_camera_link"/>
-    <child link="depth_camera_optical"/>
-  </joint>
 </robot>

Commit message: Lesson_7 Kinect V1.0

File: mark1/src/mark1_description/urdf/mark1.xacro (robot description, xacro)
@@ -137,5 +137,25 @@
       xyz="0 1 0" />
   </joint>
- <joint name="hokuyo_joint" type="fixed">
+  <!-- Hokuyo Laser -->
+  <link name="hokuyo">
+    <collision>
+      <origin xyz="0 0 0" rpy="0 0 0"/>
+      <geometry>
+    <box size="0.1 0.1 0.1"/>
+      </geometry>
+    </collision>
+    <visual>
+      <origin xyz="0 0 0" rpy="0 0 0"/>
+      <geometry>
+        <mesh filename="package://mark1/src/mark1_description/meshes/hokuyo.dae"/>
+      </geometry>
+    </visual>
+    <inertial>
+      <mass value="1e-5" />
+      <origin xyz="0 0 0" rpy="0 0 0"/>
+      <inertia ixx="1e-6" ixy="0" ixz="0" iyy="1e-6" iyz="0" izz="1e-6" />
+    </inertial>
+  </link>
+    <joint name="hokuyo_joint" type="fixed">
     <axis xyz="0 1 0" />
     <origin xyz="-0.1 0 0.19" rpy="0 0 0"/>
@@ -143,17 +163,18 @@
     <child link="hokuyo"/>
   </joint>
-  <!-- Hokuyo Laser -->
-  <link name="hokuyo">
-    <collision>
-      <origin xyz="0 0 0" rpy="0 0 0"/>
-      <geometry>
-    <box size="0.1 0.1 0.1"/>
-      </geometry>
-    </collision>
-    <visual>
-      <origin xyz="0 0 0" rpy="0 0 0"/>
-      <geometry>
-        <mesh filename="package://mark1/src/mark1_description/meshes/hokuyo.dae"/>
-      </geometry>
+  <!-- Camera -->
+  <link name="camera_link">
+    <collision>
+      <origin xyz="0 0 0" rpy="0 0 0"/>
+      <geometry>
+    <box size="0 0 0"/>
+      </geometry>
+    </collision>
+    <visual>
+      <origin xyz="0 0 0" rpy="0 0 0"/>
+      <geometry>
+    <box size="0.05 0.05  0.05"/>
+      </geometry>
+      <material name="red"/>
     </visual>
     <inertial>
@@ -163,5 +184,5 @@
     </inertial>
   </link>
-<joint name="camera_joint" type="fixed">
+  <joint name="camera_joint" type="fixed">
     <axis xyz="0 1 0" />
     <origin xyz="0.27 0 0.05" rpy="0 0  0"/>
@@ -169,10 +190,10 @@
     <child link="camera_link"/>
   </joint>
-  <!-- Camera -->
-  <link name="camera_link">
-    <collision>
-      <origin xyz="0 0 0" rpy="0 0 0"/>
-      <geometry>
-    <box size="0 0 0"/>
+    <!-- Depth Camera -->
+<link name="depth_camera_link">
+    <collision>
+      <origin xyz="0 0 0" rpy="0 0 0"/>
+      <geometry>
+    <box size="0.05 0.05 0.05"/>
       </geometry>
     </collision>
@@ -182,11 +203,25 @@
     <box size="0.05 0.05  0.05"/>
       </geometry>
-      <material name="red"/>
-    </visual>
-    <inertial>
-      <mass value="1e-5" />
+      <material name="blue"/>
+    </visual>
+    <inertial>
+      <mass value="0.210" />
       <origin xyz="0 0 0" rpy="0 0 0"/>
       <inertia ixx="1e-6" ixy="0" ixz="0" iyy="1e-6" iyz="0" izz="1e-6" />
     </inertial>
   </link>
+<joint name="depth_camera_joint" type="fixed">
+    <axis xyz="0 1 0" />
+    <origin xyz="-0.1 0 0.4" rpy="0 0  0"/>
+    <parent link="base_link"/>
+    <child link="depth_camera_link"/>
+  </joint>
+ <link name="depth_camera_optical">
+  </link>
+ <joint name="depth_camera_optical_joint" type="fixed">
+    <axis xyz="0 1 0" />
+    <origin xyz="0 0 0" rpy="-1.57 0 -1.57"/>
+    <parent link="depth_camera_link"/>
+    <child link="depth_camera_optical"/>
+  </joint>
 </robot>

Commit message: AMCL and move base is good working

File: mark1/src/mark1_description/urdf/mark1.xacro (robot description, xacro)
@@ -138,5 +138,5 @@
   </joint>
   <!-- Hokuyo Laser -->
-  <link name="hokuyo">
+  <link name="laser_link">
     <collision>
       <origin xyz="0 0 0" rpy="0 0 0"/>
@@ -161,5 +161,5 @@
     <origin xyz="-0.1 0 0.19" rpy="0 0 0"/>
     <parent link="base_link"/>
-    <child link="hokuyo"/>
+    <child link="laser_link"/>
   </joint>
   <!-- Camera -->
